Commit message: xacro and box world fixes

File: smart_arm_description/urdf/smart_arm.xacro (robot description, xacro)
@@ -33,11 +33,11 @@
 * Author: Antons Rebguns
 -->
-<robot name="rrbot" xmlns:xacro="http://www.ros.org/wiki/xacro">
-  <include filename="$(find smart_arm_description)/urdf/materials.urdf.xacro" />
-  <macro name="smart_arm" params="parent *origin">
+<robot name="smart_arm" xmlns:xacro="http://www.ros.org/wiki/xacro">
+  <xacro:include filename="$(find smart_arm_description)/urdf/materials.urdf.xacro" />
+  <xacro:macro name="smart_arm" params="parent decimated:='' *origin">
     <!-- ****** JOINT DEFINITIONS ****** -->
     <!-- Arm's base joint -->
     <joint name="arm_base_joint" type="fixed">
-      <insert_block name="origin" />
+      <xacro:insert_block name="origin" />
       <parent link="${parent}"/>
       <child link="arm_base_link"/>
@@ -119,5 +119,5 @@
         <origin xyz="0.0 0.0 0.0" rpy="0 0 0" />
         <geometry>
-          <mesh filename="package://smart_arm_description/meshes/collada/arm_base.dae"/>
+          <mesh filename="package://smart_arm_description/meshes/collada/arm_base${decimated}.dae"/>
         </geometry>
         <material name="Green" />
@@ -126,5 +126,6 @@
         <origin xyz="0.0 0.0 0.0" rpy="0 0 0" />
         <geometry>
-          <mesh filename="package://smart_arm_description/meshes/collada/arm_base.dae"/>
+          <!--box><size>0.115 0.115 0.05</size></box-->
+          <mesh filename="package://smart_arm_description/meshes/collada/arm_base${decimated}.dae"/>
         </geometry>
       </collision>
@@ -141,5 +142,5 @@
         <origin xyz="0.0 0.0 0.005" rpy="0 0 0" />
         <geometry>
-          <mesh filename="package://smart_arm_description/meshes/collada/arm_shoulder_pan.dae"/>
+          <mesh filename="package://smart_arm_description/meshes/collada/arm_shoulder_pan${decimated}.dae"/>
         </geometry>
         <material name="Grey" />
@@ -148,5 +149,5 @@
         <origin xyz="0.0 0.0 0.0" rpy="0 0 0" />
         <geometry>
-          <mesh filename="package://smart_arm_description/meshes/collada/arm_shoulder_pan.dae"/>
+          <mesh filename="package://smart_arm_description/meshes/collada/arm_shoulder_pan${decimated}.dae"/>
         </geometry>
       </collision>
@@ -163,5 +164,5 @@
         <origin xyz="0.0 0.0 0.0" rpy="0 0 0" />
         <geometry>
-          <mesh filename="package://smart_arm_description/meshes/collada/arm_shoulder_pitch.dae"/>
+          <mesh filename="package://smart_arm_description/meshes/collada/arm_shoulder_pitch${decimated}.dae"/>
         </geometry>
         <material name="Blue" />
@@ -170,5 +171,5 @@
         <origin xyz="0.0 0.0 0.0" rpy="0 0 0" />
         <geometry>
-          <mesh filename="package://smart_arm_description/meshes/collada/arm_shoulder_pitch.dae"/>
+          <mesh filename="package://smart_arm_description/meshes/collada/arm_shoulder_pitch${decimated}.dae"/>
         </geometry>
       </collision>
@@ -185,5 +186,5 @@
         <origin xyz="0.0 0.0 0.0" rpy="0 0 0" />
         <geometry>
-          <mesh filename="package://smart_arm_description/meshes/collada/arm_elbow_flex.dae"/>
+          <mesh filename="package://smart_arm_description/meshes/collada/arm_elbow_flex${decimated}.dae"/>
         </geometry>
         <material name="Green" />
@@ -192,5 +193,5 @@
         <origin xyz="0.0 0.0 0.0" rpy="0 0 0" />
         <geometry>
-          <mesh filename="package://smart_arm_description/meshes/collada/arm_elbow_flex.dae"/>
+          <mesh filename="package://smart_arm_description/meshes/collada/arm_elbow_flex${decimated}.dae"/>
         </geometry>
       </collision>
@@ -207,5 +208,5 @@
         <origin xyz="0.0 0.0 0.0" rpy="0 0 0" />
         <geometry>
-          <mesh filename="package://smart_arm_description/meshes/collada/arm_wrist_roll.dae"/>
+          <mesh filename="package://smart_arm_description/meshes/collada/arm_wrist_roll${decimated}.dae"/>
         </geometry>
         <material name="Grey" />
@@ -214,5 +215,5 @@
         <origin xyz="0.0 0.0 0.0" rpy="0 0 0" />
         <geometry>
-          <mesh filename="package://smart_arm_description/meshes/collada/arm_wrist_roll.dae"/>
+          <mesh filename="package://smart_arm_description/meshes/collada/arm_wrist_roll${decimated}.dae"/>
         </geometry>
       </collision>
@@ -229,5 +230,5 @@
         <origin xyz="0.0 0.0 0.0" rpy="0 0 0" />
         <geometry>
-          <mesh filename="package://smart_arm_description/meshes/collada/arm_right_finger.dae"/>
+          <mesh filename="package://smart_arm_description/meshes/collada/arm_right_finger${decimated}.dae"/>
         </geometry>
         <material name="Blue" />
@@ -236,5 +237,5 @@
         <origin xyz="0.0 0.0 0.0" rpy="0 0 0" />
         <geometry>
-          <mesh filename="package://smart_arm_description/meshes/collada/arm_right_finger.dae"/>
+          <mesh filename="package://smart_arm_description/meshes/collada/arm_right_finger${decimated}.dae"/>
         </geometry>
       </collision>
@@ -251,5 +252,5 @@
         <origin xyz="0.0 0.0 0.0" rpy="0 0 0" />
         <geometry>
-          <mesh filename="package://smart_arm_description/meshes/collada/arm_left_finger.dae"/>
+          <mesh filename="package://smart_arm_description/meshes/collada/arm_left_finger${decimated}.dae"/>
         </geometry>
         <material name="Green" />
@@ -258,5 +259,5 @@
         <origin xyz="0.0 0.0 0.0" rpy="0 0 0" />
         <geometry>
-          <mesh filename="package://smart_arm_description/meshes/collada/arm_left_finger.dae"/>
+          <mesh filename="package://smart_arm_description/meshes/collada/arm_left_finger${decimated}.dae"/>
         </geometry>
       </collision>
@@ -407,4 +408,4 @@
       <fudgeFactor value="1.0" />
     </gazebo>
-  </macro>
+  </xacro:macro>
 </robot>

File: smart_arm_description/urdf/smart_arm_robot.xacro (robot description, xacro)
@@ -1,9 +1,6 @@
 <?xml version="1.0"?>
-<robot name="smart_arm"
-  xmlns:sensor="http://playerstage.sourceforge.net/gazebo/xmlschema/#sensor"
-  xmlns:controller="http://playerstage.sourceforge.net/gazebo/xmlschema/#controller"
-  xmlns:interface="http://playerstage.sourceforge.net/gazebo/xmlschema/#interface">
+<robot name="smart_arm"  xmlns:xacro="http://www.ros.org/wiki/xacro">
   <!-- Included URDF Files -->
-  <include filename="$(find smart_arm_description)/urdf/smart_arm.xacro" />
+  <xacro:include filename="$(find smart_arm_description)/urdf/smart_arm.xacro" />
   <!--link name="world_link">
     <inertial>
@@ -32,5 +29,5 @@
   <!-- Used for fixing robot to Gazebo 'base_link' -->
   <link name="world"/>
-  <smart_arm parent="world">
+  <smart_arm parent="world"> <!--decimated="_decimated"-->
     <origin xyz="0 0 0" rpy="0 0 0" />
   </smart_arm>
